File: LEDController.kicad_pcb (KiCad board)
At the start: 2 copper layers, 0 parts

Commit message: Added diode and transistor
Parts:
- added J1: 3557-2, SamacSys_Parts:3557-2, F.Cu at (111.8, 55.1)
- added J10: 3557-2, SamacSys_Parts:3557-2, F.Cu at (111.8, 127.0)
- added J16: 3557-2, SamacSys_Parts:3557-2, F.Cu at (218.0, 46.0)
- added J2: 3557-2, SamacSys_Parts:3557-2, F.Cu at (112.0, 63.0)
- added J3: 3557-2, SamacSys_Parts:3557-2, F.Cu at (111.8, 71.1)
- added J4: 3557-2, SamacSys_Parts:3557-2, F.Cu at (111.8, 79.1)
- added J5: 3557-2, SamacSys_Parts:3557-2, F.Cu at (111.8, 87.1)
- added J6: 3557-2, SamacSys_Parts:3557-2, F.Cu at (111.8, 95.1)
- added J7: 3557-2, SamacSys_Parts:3557-2, F.Cu at (111.8, 103.0)
- added J8: 3557-2, SamacSys_Parts:3557-2, F.Cu at (111.8, 111.0)
- added J9: 3557-2, SamacSys_Parts:3557-2, F.Cu at (111.8, 119.0)
- added K1: J115F11CH5VDCS61.5U, SamacSys_Parts:J115F11CH5VDCS615U, F.Cu at (169.0, 72.3)
- added Q1: BCX56,135, SamacSys_Parts:PBSS4360XX, F.Cu at (197.5, 65.2)
