File: LEDController.kicad_pcb (KiCad board)
At the start: 2 copper layers, 19 parts, among them J1 3557-2, J10 3557-2, J11 TB002-500-04BE, J12 TB002-500-04BE, J16 3557-2, J17 TB002-500-04BE, J2 3557-2, J3 3557-2, J4 3557-2, J5 3557-2, J6 3557-2, J7 3557-2, J7 VP0265840000G, J8 3557-2, J9 3557-2, K1 J115F11CH5VDCS61.5U, Q1 BCX56,135

Commit message: final schematic
Parts:
- removed D2: S1M, SamacSys_Parts:DIOM5336X240N
- removed J1, J10, J16, J2, J3, J4, J5, J6, J7, J8, J9: 3557-2, SamacSys_Parts:3557-2
- removed J11, J12, J17: TB002-500-04BE, SamacSys_Parts:CONN4_TB002-500_787x299_CUD
- removed J7: VP0265840000G, SamacSys_Parts:CONN04_VP026584_20P32X18P3_AMP
- removed K1: J115F11CH5VDCS61.5U, SamacSys_Parts:J115F11CH5VDCS615U
- removed Q1: BCX56,135, SamacSys_Parts:PBSS4360XX
- removed R1: 1K, Resistor_SMD:R_0603_1608Metric_Pad0.98x0.95mm_HandSolder

Commit message: add footprints from laptop
Parts:
- added D2: S1M, SamacSys_Parts:DIOM5336X240N, F.Cu at (122.7, 94.2)
- added J1: 3557-2, SamacSys_Parts:3557-2, F.Cu at (85.3, 50.6)
- added J11: TB002-500-04BE, SamacSys_Parts:CONN4_TB002-500_787x299_CUD, F.Cu at (114.2, 86.7)
- added J12: TB002-500-04BE, SamacSys_Parts:CONN4_TB002-500_787x299_CUD, F.Cu at (114.2, 96.0)
- added J16: 3557-2, SamacSys_Parts:3557-2, F.Cu at (85.3, 106.5)
- added J17: TB002-500-04BE, SamacSys_Parts:CONN4_TB002-500_787x299_CUD, F.Cu at (114.2, 105.2)
- added J2: 3557-2, SamacSys_Parts:3557-2, F.Cu at (85.3, 58.6)
- added J3: 3557-2, SamacSys_Parts:3557-2, F.Cu at (85.3, 66.6)
- added J4: 3557-2, SamacSys_Parts:3557-2, F.Cu at (85.3, 74.6)
- added J5: 3557-2, SamacSys_Parts:3557-2, F.Cu at (85.3, 82.6)
- added J6: 3557-2, SamacSys_Parts:3557-2, F.Cu at (85.3, 90.6)
- added J8: 3557-2, SamacSys_Parts:3557-2, F.Cu at (85.3, 98.5)
- added J9: Conn_01x03_Pin, Connector_PinSocket_2.54mm:PinSocket_1x03_P2.54mm_Vertical, F.Cu at (120.9, 84.1)
- added K1: J115F11CH5VDCS61.5U, SamacSys_Parts:J115F11CH5VDCS615U, F.Cu at (115.2, 73.3)
- added Q1: BCX56,135, SamacSys_Parts:PBSS4360XX, F.Cu at (122.4, 100.8)
- added R1: 1K, Resistor_SMD:R_0603_1608Metric_Pad0.98x0.95mm_HandSolder, F.Cu at (120.7, 106.0)
