File: LEDController.kicad_pcb (KiCad board)
At the start: 2 copper layers, 16 parts, among them J1 3557-2, J11 TB002-500-04BE, J12 TB002-500-04BE, J16 3557-2, J17 TB002-500-04BE, J2 3557-2, J3 3557-2, J4 3557-2, J5 3557-2, J6 3557-2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

Commit message: wip layout
Parts:
- added C1: UVR1E102MPD, SamacSys_Parts:CAPPRD500W60D1025H2200, F.Cu at (81.6, 114.0)
- added J7: 0389690002, SamacSys_Parts:0389690002, F.Cu at (124.9, 102.0)
- moved J11 71.9 mm to (50.7, 120.6), turned to -90 degrees
- moved J17 65.8 mm to (50.7, 88.0), turned to -90 degrees
- moved J12 48.6 mm to (74.1, 123.4)
- moved J9 42.2 mm to (95.1, 117.5), turned to -90 degrees
- moved Q1 39.1 mm to (83.6, 105.5), turned to 180 degrees
- moved J8 37.8 mm to (118.2, 80.1)
- moved J16 37.7 mm to (118.2, 88.1)
- moved D2 32.7 mm to (91.6, 104.5), turned to 180 degrees
- moved J6 29.2 mm to (66.1, 112.6)
- moved J5 28.3 mm to (66.0, 103.2)
- moved K1 27.6 mm to (96.7, 93.9)
- moved J4 27.4 mm to (66.0, 94.0)
- moved J3 26.7 mm to (66.0, 85.0)
- moved R1 26.5 mm to (95.1, 113.0), turned to 90 degrees
- moved J2 26.0 mm to (66.0, 76.0)
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Connections:
- net Net-(J16-Pad2) renamed /50U
- J1 pad 2: Net-(C1-+) -> /50R
- J1 pad 4: Net-(C1-+) -> /50R
- J16 pad 1: Net-(D2-K) -> /50F
- J16 pad 3: Net-(D2-K) -> /50F
- J2 pad 2: Net-(C1-+) -> /50R
- J2 pad 4: Net-(C1-+) -> /50R
- J3 pad 2: Net-(C1-+) -> /50R
- J3 pad 4: Net-(C1-+) -> /50R
- J4 pad 2: Net-(C1-+) -> /50R
- J4 pad 4: Net-(C1-+) -> /50R
- J5 pad 2: Net-(C1-+) -> /50R
- J5 pad 4: Net-(C1-+) -> /50R
- J6 pad 2: Net-(C1-+) -> /50R
- J6 pad 4: Net-(C1-+) -> /50R
- J8 pad 1: Net-(D2-K) -> /50F
- J8 pad 3: Net-(D2-K) -> /50F
- J9 pad 2: Net-(D2-K) -> /50F
Routing:
- net Net-(D2-K): track 0.00 -> 29.1 mm
- net Net-(C1-+): track 0.00 -> 23.3 mm
- net Net-(J17-Pad1): track 0.00 -> 13.6 mm
- net Net-(J1-Pad1): track 0.00 -> 13.6 mm
- net Net-(Q1-B): track 0.00 -> 13.5 mm
- net Net-(J11-Pad4): track 0.00 -> 12.2 mm
- net Net-(J11-Pad3): track 0.00 -> 12.2 mm
- net Net-(J17-Pad2): track 0.00 -> 12.1 mm
- net Net-(J17-Pad3): track 0.00 -> 12.1 mm
- net Net-(J9-Pin_1): track 0.00 -> 3.59 mm

Commit message: wip layout
Parts:
- C1: footprint SamacSys_Parts:CAPPRD500W60D1025H2200 -> LEDController:CAPPRD500W60D1025H2200
- D2: footprint SamacSys_Parts:DIOM5336X240N -> LEDController:DIOM5336X240N
- J1, J16, J2, J3, J4, J5, J6, J8: footprint SamacSys_Parts:3557-2 -> LEDController:3557-2
- J11, J12, J17: footprint SamacSys_Parts:CONN4_TB002-500_787x299_CUD -> LEDController:CONN4_TB002-500_787x299_CUD
- J7: footprint SamacSys_Parts:0389690002 -> LEDController:0389690002
- K1: footprint SamacSys_Parts:J115F11CH5VDCS615U -> LEDController:J115F11CH5VDCS615U
- Q1: footprint SamacSys_Parts:PBSS4360XX -> LEDController:PBSS4360XX
- moved D2 6.86 mm to (98.5, 104.6)
- moved Q1 6.86 mm to (90.4, 105.6)
- moved J9 3.73 mm to (95.5, 113.8)
- moved R1 3.73 mm to (95.5, 109.3)
- moved C1 0.88 mm to (81.2, 114.8)
Connections:
- D2 pad 1: Net-(D2-K) -> /50F
- D2 pad 2: Net-(C1-+) -> Net-(D2-A)
- K1 pad 1: Net-(D2-K) -> /50F
- K1 pad 2: Net-(C1-+) -> Net-(D2-A)
- K1 pad 3: Net-(C1-+) -> /50R
- K1 pad 5: Net-(D2-K) -> /50F
- Q1 pad 2: Net-(C1-+) -> Net-(D2-A)
- Q1 pad 4: Net-(C1-+) -> Net-(D2-A)
Routing:
- net /50F: track 0.00 -> 30.5 mm
- net Net-(D2-K): track 29.1 -> 0.00 mm
- net Net-(D2-A): track 0.00 -> 28.5 mm
- net Net-(C1-+): track 23.3 -> 0.00 mm
- net GND: track 0.00 -> 10.7 mm
- net Net-(Q1-B): track 13.5 -> 7.69 mm
- added copper zone on B.Cu, net /50F
- added copper zone on F.Cu, net /50F
- added copper zone on B.Cu, net /50R
- added copper zone on F.Cu, net /50R
- added copper zone on B.Cu, net /50U
- added copper zone on F.Cu, net /50U
- added copper zone on B.Cu, net GND
- added copper zone on F.Cu, net GND
Other:
- board outline added: 88 x 67.5 mm

Commit message: Final Layout
Parts:
- C1: footprint LEDController:CAPPRD500W60D1025H2200 -> Footprints:CAPPRD500W60D1025H2200
- D2: footprint LEDController:DIOM5336X240N -> Footprints:DIOM5336X240N
- J1, J16, J2, J3, J4, J5, J6, J8: footprint LEDController:3557-2 -> Footprints:3557-2
- J11, J12, J17: footprint LEDController:CONN4_TB002-500_787x299_CUD -> Footprints:CONN4_TB002-500_787x299_CUD
- J7: footprint LEDController:0389690002 -> Footprints:0389690002
- K1: footprint LEDController:J115F11CH5VDCS615U -> Footprints:J115F11CH5VDCS615U
- Q1: footprint LEDController:PBSS4360XX -> Footprints:PBSS4360XX
- moved C1 1.50 mm to (82.7, 114.8)
Routing:
- net Net-(J17-Pad1): track 13.6 -> 27.2 mm
- net Net-(J1-Pad1): track 13.6 -> 27.2 mm
- net Net-(J11-Pad4): track 12.2 -> 24.5 mm
- net Net-(J11-Pad3): track 12.2 -> 24.3 mm
- net Net-(J17-Pad2): track 12.1 -> 24.2 mm
- net Net-(J17-Pad3): track 12.1 -> 24.1 mm
- net /50F: track 30.5 -> 32.8 mm
Other:
- outline, holes or cut-outs redrawn
