File: LEDControllerPDB/5VRegulator.kicad_sch (KiCad schematic)
At the start: 9 parts

Commit message: add name
Other:
- title: (none) -> 5V Regulator
Changed lines of the file:
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@@
 	(generator_version "9.0")
 	(paper "A4")
+	(title_block
+		(title "5V Regulator")
+		(date "2025-04-18")
+		(rev "01")
+	)
 	(junction
 		(at 140.97 96.52)

Commit message: fix regulator
Connections:
- net Vin: now also CR1.6 (VCC)
- net Vout: no longer R3.1
- net at CR1.5 (CII), R2.1: now also R3.1
Other:
- moved on the sheet: C1, C2, R2, R3, Rsc1
