File: LEDControllerPDB/LEDController.kicad_pcb (KiCad board)
At the start: 2 copper layers, 99.7 x 73.9 mm, 21 parts, among them J1 3557-2, J11 TB002-500-04BE, J12 TB002-500-04BE, J17 TB002-500-04BE, J2 3557-2, J3 3557-2, J4 3557-2, J5 3557-2, J6 3557-2, J7 0389690002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

Commit message: add 24v support and reverse voltage protection
Parts:
- added C1: 470uF, LEDController:CAPPRD500W60D1000H1350, F.Cu at (156.8, 81.7)
- added C2: 100uF, Capacitor_THT:CP_Radial_D5.0mm_P2.50mm, F.Cu at (173.1, 94.8)
- added C3: 470pF, Capacitor_SMD:C_0603_1608Metric_Pad1.08x0.95mm_HandSolder, F.Cu at (169.6, 65.5)
- added CR1: MC34063ABD-TR, LEDController:SO-8_STM, F.Cu at (169.2, 79.5)
- added CR2: SMD110PL-TP, LEDController:SOD-123FL_MCC, F.Cu at (167.9, 84.6)
- added D1: D_Zener, Diode_SMD:D_SOD-123, F.Cu at (163.7, 96.5)
- added L1: SDR1105-201KL, LEDController:IND_BOURNS_SDR1105, F.Cu at (160.6, 70.2)
- added Q1: DMP3099L, Package_TO_SOT_SMD:SOT-23-3, F.Cu at (163.3, 100.6)
- added R2: 3.6k, Resistor_SMD:R_0603_1608Metric_Pad0.98x0.95mm_HandSolder, F.Cu at (179.8, 92.8)
- added R3: 1.2k, Resistor_SMD:R_0603_1608Metric_Pad0.98x0.95mm_HandSolder, F.Cu at (179.8, 95.3)
- added R4: R470, Resistor_SMD:R_0201_0603Metric_Pad0.64x0.40mm_HandSolder, F.Cu at (167.3, 99.1)
- added Rsc1: .33, Resistor_SMD:R_0603_1608Metric_Pad0.98x0.95mm_HandSolder, F.Cu at (169.6, 68.0)
- R1: footprint Resistor_THT:R_Axial_DIN0309_L9.0mm_D3.2mm_P12.70mm_Horizontal -> Resistor_SMD:R_0603_1608Metric_Pad0.98x0.95mm_HandSolder
- renumbered C1 to C4
Connections:
- D2 pad 1: /50F -> /5V
- J9 pad 2: /50F -> /5V
- K1 pad 1: /50F -> /5V

Commit message: rerout
Parts:
- removed D2: 1N4007, Diode_THT:D_DO-41_SOD81_P10.16mm_Horizontal
- removed J8: 3557-2, LEDController:FUSE_3555-2
- removed Q2: PN2222ATA, LEDController:TO-92_ONS
- removed REF** (x4): MountingHole_5mm, MountingHole:MountingHole_5mm
- added CR3: S1G-E3/61T, LEDController:DIODE_DO214AC, F.Cu at (90.5, 104.6)
- added J10: 3557-2, LEDController:3557-2, F.Cu at (116.7, 67.1)
- added Q3: MMBT2222A, Package_TO_SOT_SMD:SOT-23, F.Cu at (92.2, 109.1)
- R4: value R470 -> 470
- moved L1 62.5 mm to (113.2, 111.1), turned to 180 degrees
- moved CR2 62.0 mm to (125.1, 129.4)
- moved Q1 62.0 mm to (120.5, 145.4)
- moved D1 62.0 mm to (120.9, 141.4)
- moved R2 62.0 mm to (137.0, 137.7)
- moved R3 62.0 mm to (137.0, 140.2)
- moved R4 62.0 mm to (124.5, 143.9)
- moved C1 62.0 mm to (114.0, 126.6)
- moved C2 62.0 mm to (130.3, 139.7)
- moved CR1 62.0 mm to (126.4, 124.3)
- moved Rsc1 62.0 mm to (126.7, 112.9)
- moved C3 54.6 mm to (131.4, 104.6)
- moved J7 30.6 mm to (125.4, 80.5)
Connections:
- J11 pad 2: GND -> Net-(J11-Pad2)
- J11 pad 3: Net-(J11-Pad3) -> GND
- J12 pad 2: GND -> Net-(J12-Pad2)
- J12 pad 4: GND -> Net-(J12-Pad4)
- J17 pad 1: Net-(J17-Pad1) -> GND
- J17 pad 3: Net-(J17-Pad3) -> GND
- J2 pad 1: Net-(J17-Pad3) -> Net-(J17-Pad2)
- J2 pad 3: Net-(J17-Pad3) -> Net-(J17-Pad2)
- J3 pad 1: Net-(J17-Pad2) -> Net-(J11-Pad4)
- J3 pad 3: Net-(J17-Pad2) -> Net-(J11-Pad4)
- J4 pad 1: Net-(J17-Pad1) -> Net-(J11-Pad2)
- J4 pad 3: Net-(J17-Pad1) -> Net-(J11-Pad2)
- J5 pad 1: Net-(J11-Pad4) -> Net-(J12-Pad4)
- J5 pad 3: Net-(J11-Pad4) -> Net-(J12-Pad4)
- J6 pad 1: Net-(J11-Pad3) -> Net-(J12-Pad2)
- J6 pad 3: Net-(J11-Pad3) -> Net-(J12-Pad2)
- J9 pad 1: GND -> /5V
- J9 pad 2: /5V -> GND
Routing:
- net Net-(J11-Pad3): track 27.8 -> 0.00 mm
- net Net-(J1-Pad1): track 27.2 -> 0.00 mm
- net Net-(J17-Pad1): track 27.2 -> 0.00 mm
- net Net-(J11-Pad4): track 24.2 -> 0.00 mm
- net Net-(J17-Pad2): track 24.2 -> 0.00 mm
- net Net-(J17-Pad3): track 24.1 -> 0.00 mm
- net Net-(Q3-B): track 5.72 -> 0.00 mm
- net (no net): track 0.00 -> 5.72 mm

Commit message: finished pdb
Parts:
- added M2.5 / #6: MountingHole_2.7mm_M2.5, MountingHole:MountingHole_2.7mm_M2.5, F.Cu at (52.0, 43.0)
- added REF**: MountingHole_2.7mm_M2.5, MountingHole:MountingHole_2.7mm_M2.5, F.Cu at (52.0, 114.7)
- added REF**: MountingHole_2.7mm_M2.5, MountingHole:MountingHole_2.7mm_M2.5, F.Cu at (129.0, 114.7)
- added REF**: MountingHole_2.7mm_M2.5, MountingHole:MountingHole_2.7mm_M2.5, F.Cu at (129.0, 43.0)
- R4: footprint Resistor_SMD:R_0201_0603Metric_Pad0.64x0.40mm_HandSolder -> Resistor_SMD:R_0603_1608Metric_Pad0.98x0.95mm_HandSolder
- moved R4 53.6 mm to (94.2, 99.8), turned to 180 degrees
- moved Q1 51.7 mm to (98.2, 98.8), turned to 90 degrees
- moved C2 44.4 mm to (99.7, 107.5), turned to -90 degrees
- moved D1 44.3 mm to (98.2, 103.3), turned to 180 degrees
- moved CR2 41.2 mm to (101.7, 95.5), turned to 180 degrees
- moved R3 38.3 mm to (116.2, 108.0), turned to 180 degrees
- moved R2 37.9 mm to (116.2, 106.0)
- moved R1 28.2 mm to (90.7, 97.8)
- moved C4 27.7 mm to (80.5, 91.0)
- moved J11 26.8 mm to (48.5, 93.7)
- moved C3 26.7 mm to (104.7, 104.5), turned to 180 degrees
- moved CR1 25.7 mm to (110.7, 104.0)
- moved Rsc1 24.6 mm to (104.7, 102.0)
- moved J6 23.2 mm to (71.1, 94.2), turned to 90 degrees
- moved C1 22.3 mm to (122.5, 106.0), turned to 90 degrees
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Routing:
- net /5V: track 0.00 -> 95.2 mm, vias 0 -> 4
- net Net-(J11-Pad2): track 0.00 -> 28.9 mm
- net Net-(J11-Pad4): track 0.00 -> 28.1 mm
- net Net-(J12-Pad2): track 0.00 -> 26.7 mm
- net Net-(J12-Pad4): track 0.00 -> 26.2 mm
- net Net-(J17-Pad2): track 0.00 -> 25.2 mm
- net Net-(J1-Pad1): track 0.00 -> 24.4 mm
- net /5VReg/Vin: track 0.00 -> 14.2 mm
- net Net-(CR1-SWE): track 0.00 -> 13.8 mm, vias 0 -> 2
- net /50F: track 40.5 -> 29.9 mm, vias 0 -> 2
- net Net-(CR1-DRC): track 0.00 -> 9.00 mm
- net Net-(J9-Pin_3): track 6.37 -> 13.9 mm, vias 0 -> 2
- net (no net): track 5.72 -> 0.00 mm
- net Net-(D1-A): track 0.00 -> 5.44 mm
- net Net-(K1-COIL_2): track 18.7 -> 22.8 mm
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Other:
- board size 99.7 x 73.9 mm -> 104 x 79.1 mm
- board text added: "+"
- board text added: "-"
- board text added: "12-24V"
- board text added: "5v"
- board text added: "A"
- board text added: "B"
- board text added: "Main Fuse. 30A Max"
- board text added: "Output Fuses. 10A Max"
- board text removed: "Vcc"

Commit message: done
Parts:
- removed J9: Conn_01x03_Pin, Connector_PinSocket_2.54mm:PinSocket_1x03_P2.54mm_Vertical
- removed R1: 1K, Resistor_SMD:R_0603_1608Metric_Pad0.98x0.95mm_HandSolder
- added J13: 647676-3, LEDController:TE_647676-3, F.Cu at (83.8, 102.9)
- added J8: HB9500-9.5-2P, LEDController:SHDR2W140P0X950_1X2_2055X1800X1440P, F.Cu at (108.4, 60.0)
- J7: value 0389690002 -> Conn_02x02_Row_Letter_First; footprint LEDController:0389690002 -> Connector_PinHeader_2.54mm:PinHeader_2x02_P2.54mm_Vertical
- moved J7 45.4 mm to (85.2, 93.2), turned to 0 degrees
- moved J3 8.02 mm to (61.5, 63.2)
- moved C2 8.02 mm to (97.8, 99.7)
- moved C3 8.02 mm to (102.8, 96.7)
- moved CR1 8.02 mm to (108.8, 96.2)
- moved CR2 8.02 mm to (99.8, 87.7)
- moved CR3 8.02 mm to (93.8, 85.5)
- moved D1 8.02 mm to (96.3, 95.5)
- moved L1 8.02 mm to (108.8, 87.7)
- moved Q1 8.02 mm to (96.3, 91.0)
- moved Q3 8.02 mm to (87.8, 85.5)
- moved R2 8.02 mm to (114.3, 98.2)
- moved R3 8.02 mm to (114.3, 100.2)
- moved R4 8.02 mm to (92.3, 92.0)
- moved Rsc1 8.02 mm to (102.8, 94.2)
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Connections:
- D1 pad 1: /5VReg/Vin -> Net-(D1-K)
- J7 pad 1: /50U -> Net-(D1-K)
- J7 pad 2: GND -> Net-(D1-K)
- Q1 pad 2: /5VReg/Vin -> Net-(D1-K)
- Q3 pad 1: Net-(Q3-B) -> /Relay Controll
Routing:
- net /Relay Controll: track 0.00 -> 21.1 mm, vias 0 -> 2
- net Net-(D1-K): track 0.00 -> 18.1 mm
- net Net-(J9-Pin_3): track 13.9 -> 0.00 mm, vias 2 -> 0
- net /5V: track 95.2 -> 100.7 mm, vias 4 -> 3
- net /5VReg/Vin: track 14.2 -> 19.0 mm
- net Net-(Q3-B): track 2.66 -> 0.00 mm
Other:
- board size 104 x 79.1 mm -> 97.5 x 84.4 mm
- board text added: "12V 24V"
- board text added: "5V"
- board text added: "Supply Select"

Commit message: fix regulator
Parts:
- moved C3 0.15 mm to (102.8, 96.8)
- turned R3 to 0 degrees
Connections:
- CR1 pad 6: unconnected-(CR1-VCC-Pad6) -> /5VReg/Vin
- R3 pad 1: /5V -> Net-(CR1-CII)
Routing:
- net /5VReg/Vin: track 19.0 -> 34.8 mm
- net Net-(CR1-CII): track 2.16 -> 4.16 mm
- net /5V: track 100.7 -> 98.7 mm
